File: ergogen/pcbs/temporal_back_plate_small.kicad_pcb (KiCad board)
At the start: 2 copper layers, 127.5 x 91.9 mm, 5 parts

Commit message: add some graphics
Parts:
- added ?: , utility_circle, F.Cu at (129.3, 72.0)
Changed lines of the file:
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@@
+    )
+  )
+  (footprint "utility_circle" (layer "F.Cu")
+    (at 129.2922032 72.02066630000002 0)
+    (fp_circle
+      (center 0 0)
+      (end 30 0)
+      (stroke (width 0.5) (type dash))
+      (fill none)
+      (layer "F.SilkS")
+    )
+    (fp_circle
+      (center 0 0)
+      (end 30 0)
+      (stroke (width 0.5) (type dash))
+      (fill none)
+      (layer "B.SilkS")
     )
   )
