File: ergogen/output/pcbs/mcu_cover.kicad_pcb (KiCad board)
At the start: 2 copper layers, 20.2 x 58.7 mm, 2 parts

Commit message: folder cleanup
Changed lines of the file:
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@@
   (title_block
     (title "mcu_cover")
-    (date "2025-11-12")
+    (date "2025-11-16")
     (rev "1")
     (company "curtis bollinger")
@@
     )
   )
-  (gr_line (start 166.73162046604247 95.65746366006574) (end 166.73162046604247 41.9845974) (layer Edge.Cuts) (stroke (width 0.15) (type default)))
-(gr_line (start 164.23162046604247 39.4845974) (end 149.05712050000002 39.4845974) (layer Edge.Cuts) (stroke (width 0.15) (type default)))
+  (gr_line (start 166.73162050000002 95.65746367967114) (end 166.73162050000002 41.9845974) (layer Edge.Cuts) (stroke (width 0.15) (type default)))
+(gr_line (start 164.23162050000002 39.4845974) (end 149.05712050000002 39.4845974) (layer Edge.Cuts) (stroke (width 0.15) (type default)))
 (gr_line (start 146.55712050000002 86.89647361252233) (end 146.55712050000002 41.9845974) (layer Edge.Cuts) (stroke (width 0.15) (type default)))
-(gr_line (start 147.8071205 89.06153711252233) (end 156.9341933799224 94.33105509502951) (layer Edge.Cuts) (stroke (width 0.15) (type default)))
+(gr_line (start 147.8071205 89.06153711252232) (end 156.93419337992236 94.33105509502948) (layer Edge.Cuts) (stroke (width 0.15) (type default)))
+(gr_line (start 162.98162049826797 97.82252717867114) (end 156.9341984 94.33104639999999) (layer Edge.Cuts) (stroke (width 0.15) (type default)))
+(gr_arc (start 166.73162050000002 41.9845974) (mid 165.9993875 40.2168304) (end 164.23162050000002 39.4845974) (layer Edge.Cuts) (stroke (width 0.15) (type default)))
+(gr_arc (start 149.05712050000002 39.4845974) (mid 147.28935350000003 40.2168304) (end 146.55712050000002 41.9845974) (layer Edge.Cuts) (stroke (width 0.15) (type default)))
 (gr_arc (start 146.55712050000002 86.89647361252233) (mid 146.89205700000002 88.14647361252233) (end 147.80712050000002 89.06153711252233) (layer Edge.Cuts) (stroke (width 0.15) (type default)))
-(gr_line (start 162.9816204643104 97.82252715906573) (end 156.9341984 94.33104639999999) (layer Edge.Cuts) (stroke (width 0.15) (type default)))
-(gr_arc (start 166.73162046604247 41.9845974) (mid 165.99938746604246 40.2168304) (end 164.23162046604247 39.4845974) (layer Edge.Cuts) (stroke (width 0.15) (type default)))
-(gr_arc (start 149.05712050000002 39.4845974) (mid 147.28935350000003 40.2168304) (end 146.55712050000002 41.9845974) (layer Edge.Cuts) (stroke (width 0.15) (type default)))
-(gr_arc (start 162.98162046604247 97.82252716006575) (mid 165.48162046604247 97.82252716006575) (end 166.73162046604247 95.65746366006574) (layer Edge.Cuts) (stroke (width 0.15) (type default)))
+(gr_arc (start 162.98162050000002 97.82252717967114) (mid 165.48162050000002 97.82252717967114) (end 166.73162050000002 95.65746367967114) (layer Edge.Cuts) (stroke (width 0.15) (type default)))
 (gr_line (start 151.12162050000003 73.7845974) (end 161.44162050000003 73.7845974) (layer Edge.Cuts) (stroke (width 0.15) (type default)))
 (gr_line (start 161.68162050000004 73.5445974) (end 161.68162050000004 48.7245974) (layer Edge.Cuts) (stroke (width 0.15) (type default)))
 (gr_line (start 161.44162050000003 48.4845974) (end 151.12162050000003 48.4845974) (layer Edge.Cuts) (stroke (width 0.15) (type default)))
 (gr_line (start 150.88162050000003 48.7245974) (end 150.88162050000003 73.5445974) (layer Edge.Cuts) (stroke (width 0.15) (type default)))
-(gr_arc (start 162.98162046604247 97.82252716006575) (mid 162.98162046604247 97.82252716006575) (end 162.98162046604247 97.82252716006575) (layer Edge.Cuts) (stroke (width 0.15) (type default)))
+(gr_arc (start 162.98162050000002 97.82252717967114) (mid 162.98162050000002 97.82252717967114) (end 162.98162050000002 97.82252717967114) (layer Edge.Cuts) (stroke (width 0.15) (type default)))
 (gr_arc (start 161.44162050000003 73.7845974) (mid 161.6113261 73.714303) (end 161.68162050000004 73.5445974) (layer Edge.Cuts) (stroke (width 0.15) (type default)))
 (gr_arc (start 161.68162050000004 48.7245974) (mid 161.6113261 48.5548918) (end 161.44162050000003 48.4845974) (layer Edge.Cuts) (stroke (width 0.15) (type default)))
