File: pcbs/back_plate_38/back_plate_38.kicad_pcb (KiCad board)
At the start: 2 copper layers, 117.6 x 95.3 mm, 6 parts

Commit message: update generated files
Parts:
- moved G1 48.7 mm to (108.4, 63.0), turned to 0 degrees
- moved MH3 0.34 mm to (143.2, 97.7)
- moved MH4 0.34 mm to (104.3, 92.5)
- moved MH5 0.34 mm to (73.5, 78.3)
- moved MH1 0.34 mm to (90.4, 47.0)
- moved MH2 0.34 mm to (127.1, 46.0)
Other:
- outline, holes or cut-outs redrawn

Commit message: update generated files
Parts:
- moved MH3 0.45 mm to (142.8, 97.7)
- moved MH4 0.45 mm to (103.9, 92.5)
Other:
- outline, holes or cut-outs redrawn
