File: pcbs/mcu_cover/mcu_cover.kicad_pcb (KiCad board)
At the start: 2 copper layers, 19.4 x 56.4 mm, 2 parts

Commit message: update gen files
Parts:
- moved MH1 136.0 mm to (259.9, 167.4)
- moved MH2 136.0 mm to (273.5, 175.3)
Changed lines of the file:
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@@
 	(title_block
 		(title "mcu_cover")
-		(date "2026-01-18")
+		(date "2026-01-22")
 		(rev "1")
 		(company "Curtis Bollinger")
@@
 	(footprint "ceoloide:mounting_hole_npth"
 		(layer "F.Cu")
-		(at 149.939872 87.435966)
-		(property "Reference" "MH1"
+		(at 273.539872 175.289966)
+		(property "Reference" "MH2"
 			(at 0 2.55 0)
 			(layer "F.SilkS")
@@
 	(footprint "ceoloide:mounting_hole_npth"
 		(layer "F.Cu")
-		(at 163.539872 95.289966)
-		(property "Reference" "MH2"
+		(at 259.939872 167.435966)
+		(property "Reference" "MH1"
 			(at 0 2.55 0)
 			(layer "F.SilkS")
@@
 		(embedded_fonts no)
 	)
-	(gr_arc
-		(start 162.389872 75.785966)
-		(mid 162.302014 75.99811)
-		(end 162.089872 76.085966)
-		(stroke
-			(width 0.15)
-			(type default)
-		)
-		(layer "Edge.Cuts")
-	)
-	(gr_line
-		(start 147.015372 87.427292)
-		(end 147.015372 44.760966)
-		(stroke
-			(width 0.15)
-			(type default)
-		)
-		(layer "Edge.Cuts")
-	)
-	(gr_arc
-		(start 148.490372 89.982067)
-		(mid 147.41061 88.902288)
-		(end 147.015372 87.427292)
-		(stroke
-			(width 0.15)
-			(type default)
-		)
-		(layer "Edge.Cuts")
-	)
-	(gr_arc
-		(start 162.089872 50.285966)
-		(mid 162.302034 50.373822)
-		(end 162.389872 50.585966)
-		(stroke
-			(width 0.15)
-			(type default)
-		)
-		(layer "Edge.Cuts")
-	)
-	(gr_line
-		(start 163.514872 41.810966)
-		(end 149.965372 41.810966)
-		(stroke
-			(width 0.15)
-			(type default)
-		)
-		(layer "Edge.Cuts")
-	)
-	(gr_arc
-		(start 147.015372 44.760966)
-		(mid 147.879417 42.675013)
-		(end 149.965372 41.810966)
+	(gr_line
+		(start 272.389872 155.785966)
+		(end 272.389872 130.585966)
+		(stroke
+			(width 0.15)
+			(type default)
+		)
+		(layer "Edge.Cuts")
+	)
+	(gr_arc
+		(start 261.089872 130.585966)
+		(mid 261.17775 130.373846)
+		(end 261.389872 130.285966)
+		(stroke
+			(width 0.15)
+			(type default)
+		)
+		(layer "Edge.Cuts")
+	)
+	(gr_arc
+		(start 276.464872 175.249984)
+		(mid 274.989898 177.804864)
+		(end 272.039872 177.804759)
+		(stroke
+			(width 0.15)
+			(type default)
+		)
+		(layer "Edge.Cuts")
+	)
+	(gr_arc
+		(start 273.514872 121.810966)
+		(mid 275.600867 122.674989)
+		(end 276.464872 124.760966)
+		(stroke
+			(width 0.15)
+			(type default)
+		)
+		(layer "Edge.Cuts")
+	)
+	(gr_line
+		(start 257.015372 167.427292)
+		(end 257.015372 124.760966)
+		(stroke
+			(width 0.15)
+			(type default)
+		)
+		(layer "Edge.Cuts")
+	)
+	(gr_line
+		(start 273.514872 121.810966)
+		(end 259.965372 121.810966)
+		(stroke
+			(width 0.15)
+			(type default)
+		)
+		(layer "Edge.Cuts")
+	)
+	(gr_line
+		(start 261.089872 130.585966)
+		(end 261.089872 155.785966)
+		(stroke
+			(width 0.15)
+			(type default)
+		)
+		(layer "Edge.Cuts")
+	)
+	(gr_arc
+		(start 272.389872 155.785966)
+		(mid 272.302014 155.99811)
+		(end 272.089872 156.085966)
+		(stroke
+			(width 0.15)
+			(type default)
+		)
+		(layer "Edge.Cuts")
+	)
+	(gr_arc
+		(start 257.015372 124.760966)
+		(mid 257.879417 122.675013)
+		(end 259.965372 121.810966)
+		(stroke
+			(width 0.15)
+			(type default)
+		)
+		(layer "Edge.Cuts")
+	)
+	(gr_line
+		(start 272.089872 130.285966)
+		(end 261.389872 130.285966)
+		(stroke
+			(width 0.15)
+			(type default)
+		)
+		(layer "Edge.Cuts")
+	)
+	(gr_line
+		(start 276.464872 175.249984)
+		(end 276.464872 124.760966)
+		(stroke
+			(width 0.15)
+			(type default)
+		)
+		(layer "Edge.Cuts")
+	)
+	(gr_line
+		(start 272.039872 177.804759)
+		(end 260.343677 171.051957)
 		(stroke
 			(width 0.15)
@@
 	)
 	(gr_circle
-		(center 149.939872 87.435966)
-		(end 150.939872 87.435966)
+		(center 259.939872 167.435966)
+		(end 260.939872 167.435966)
 		(stroke
 			(width 0.15)
@@
 		(layer "Edge.Cuts")
 	)
-	(gr_arc
-		(start 151.389872 76.085966)
-		(mid 151.17777 75.998086)
-		(end 151.089872 75.785966)
-		(stroke
-			(width 0.15)
-			(type default)
-		)
-		(layer "Edge.Cuts")
-	)
-	(gr_arc
-		(start 163.514872 41.810966)
-		(mid 165.600867 42.674989)
-		(end 166.464872 44.760966)
-		(stroke
-			(width 0.15)
-			(type default)
-		)
-		(layer "Edge.Cuts")
-	)
-	(gr_line
-		(start 166.464872 95.249984)
-		(end 166.464872 44.760966)
-		(stroke
-			(width 0.15)
-			(type default)
-		)
-		(layer "Edge.Cuts")
-	)
-	(gr_line
-		(start 162.039872 97.804759)
-		(end 150.343677 91.051957)
-		(stroke
-			(width 0.15)
-			(type default)
-		)
-		(layer "Edge.Cuts")
-	)
-	(gr_line
-		(start 151.089872 50.585966)
-		(end 151.089872 75.785966)
-		(stroke
-			(width 0.15)
-			(type default)
-		)
-		(layer "Edge.Cuts")
-	)
-	(gr_arc
-		(start 151.089872 50.585966)
-		(mid 151.17775 50.373846)
-		(end 151.389872 50.285966)
-		(stroke
-			(width 0.15)
-			(type default)
-		)
-		(layer "Edge.Cuts")
-	)
-	(gr_line
-		(start 162.089872 50.285966)
-		(end 151.389872 50.285966)
-		(stroke
-			(width 0.15)
-			(type default)
-		)
-		(layer "Edge.Cuts")
-	)
-	(gr_arc
-		(start 166.464872 95.249984)
-		(mid 164.989898 97.804864)
-		(end 162.039872 97.804759)
-		(stroke
-			(width 0.15)
-			(type default)
-		)
-		(layer "Edge.Cuts")
-	)
-	(gr_line
-		(start 151.389872 76.085966)
-		(end 162.089872 76.085966)
+	(gr_line
+		(start 258.490372 169.982067)
+		(end 260.343627 171.052044)
 		(stroke
 			(width 0.15)
@@
 	)
 	(gr_circle
-		(center 163.539872 95.289966)
-		(end 164.539872 95.289966)
+		(center 273.539872 175.289966)
+		(end 274.539872 175.289966)
 		(stroke
 			(width 0.15)
@@
 		(layer "Edge.Cuts")
 	)
-	(gr_line
-		(start 162.389872 75.785966)
-		(end 162.389872 50.585966)
-		(stroke
-			(width 0.15)
-			(type default)
-		)
-		(layer "Edge.Cuts")
-	)
-	(gr_line
-		(start 148.490372 89.982067)
-		(end 150.343627 91.052044)
+	(gr_arc
+		(start 261.389872 156.085966)
+		(mid 261.17777 155.998086)
+		(end 261.089872 155.785966)
+		(stroke
+			(width 0.15)
+			(type default)
+		)
+		(layer "Edge.Cuts")
+	)
+	(gr_arc
+		(start 258.490372 169.982067)
+		(mid 257.41061 168.902288)
+		(end 257.015372 167.427292)
+		(stroke
+			(width 0.15)
+			(type default)
+		)
+		(layer "Edge.Cuts")
+	)
+	(gr_arc
+		(start 272.089872 130.285966)
+		(mid 272.302034 130.373822)
+		(end 272.389872 130.585966)
+		(stroke
+			(width 0.15)
+			(type default)
+		)
+		(layer "Edge.Cuts")
+	)
+	(gr_line
+		(start 261.389872 156.085966)
+		(end 272.089872 156.085966)
 		(stroke
 			(width 0.15)
@@
 		(polygon
 			(pts
-				(xy 145.015372 39.810966) (xy 168.464872 39.810966) (xy 168.464872 99.804759) (xy 145.015372 99.804759)
+				(xy 255.015372 119.810966) (xy 278.464872 119.810966) (xy 278.464872 179.804759) (xy 255.015372 179.804759)
 			)
 		)
@@
 		(polygon
 			(pts
-				(xy 145.015372 39.810966) (xy 168.464872 39.810966) (xy 168.464872 99.804759) (xy 145.015372 99.804759)
-			)
-		)
+				(xy 255.015372 119.810966) (xy 278.464872 119.810966) (xy 278.464872 179.804759) (xy 255.015372 179.804759)
+			)
+		)
