File: pcbs/top_plate_40/top_plate_40.kicad_pcb (KiCad board)
At the start: 2 copper layers, 131.6 x 107.9 mm, 6 parts

Commit message: update generated files
Parts:
- moved MH3 19.7 mm to (160.5, 107.7), turned to -30 degrees
- moved G1 0.34 mm to (92.8, 83.0), turned to 0 degrees
- moved MH4 0.34 mm to (104.3, 92.5)
- moved MH5 0.34 mm to (73.5, 78.3)
- moved MH1 0.34 mm to (90.4, 47.0)
- moved MH2 0.34 mm to (127.1, 46.0)
Other:
- outline, holes or cut-outs redrawn

Commit message: update generated files
Parts:
- moved MH3 0.45 mm to (160.0, 107.7)
- moved MH4 0.45 mm to (103.9, 92.5)
Other:
- board size 131.6 x 107.9 mm -> 131.2 x 107.9 mm
