File: pcbs/top_plate_42/top_plate_42.kicad_pcb (KiCad board)
At the start: 2 copper layers, 131.8 x 95.3 mm, 6 parts

Commit message: update generated files
Parts:
- moved MH5 20.2 mm to (54.1, 73.4), turned to 10 degrees
- moved G1 0.34 mm to (92.8, 83.0), turned to 0 degrees
- moved MH3 0.34 mm to (143.2, 97.7)
- moved MH4 0.34 mm to (104.3, 92.5)
- moved MH1 0.34 mm to (90.4, 47.0)
- moved MH2 0.34 mm to (127.1, 46.0)
Other:
- outline, holes or cut-outs redrawn

Commit message: update generated files
Parts:
- moved MH3 0.45 mm to (142.8, 97.7)
- moved MH4 0.45 mm to (103.9, 92.5)
Other:
- board size 131.8 x 95.3 mm -> 131.3 x 95.3 mm
