File: pcbs/top_plate_42/top_plate_42.kicad_pcb (KiCad board)
At the start: 2 copper layers, 140.4 x 101.6 mm, 5 parts

Commit message: update gen files
Parts:
- moved MH2 136.0 mm to (237.6, 126.6)
- moved MH3 136.0 mm to (264.0, 184.8)
- moved MH1 136.0 mm to (201.1, 120.6)
- moved MH4 136.0 mm to (227.4, 169.6)
- moved MH5 136.0 mm to (164.6, 153.5)
Other:
- outline, holes or cut-outs redrawn
